File: tool-lockers-pcb.sch (KiCad schematic (older format))
At the start: 16 parts, among them J1 LOCK, J2 POWER, J3 BUTTON, J4 LED, Q1 Q_NMOS_GSD, SW1 SW_Push, U1 R-78E5.0-1.0, U2 WeMos_D1_mini

Commit message: Fix MOSFET footprint and add thermal zone
Parts:
- removed Q1: Q_NMOS_GSD, Package_TO_SOT_SMD:TO-252-3_TabPin2, symbol Device:Q_NMOS_GSD
- added Q1: Q_NMOS_GDS, Package_TO_SOT_SMD:TO-252-3_TabPin2, symbol Device:Q_NMOS_GDS
Connections:
- net GND: now also Q1.3 (S)
- net LOCK_RELEASE: now also Q1.2 (D)
- net LOCK_RELEASE_SIGNAL: now also Q1.1 (G)
Changed lines of the file:
@@
 Text Label 8550 4300 0    50   ~ 0
 SPEAKER
-$Comp
-L Device:Q_NMOS_GSD Q1
-U 1 1 5D25B437
-P 5250 6150
-F 0 "Q1" H 5456 6196 50  0000 L CNN
-F 1 "Q_NMOS_GSD" H 5456 6105 50  0000 L CNN
-F 2 "Package_TO_SOT_SMD:TO-252-3_TabPin2" H 5450 6250 50  0001 C CNN
-F 3 "~" H 5250 6150 50  0001 C CNN
-	1    5250 6150
-	1    0    0    -1
-$EndComp
 Text Label 5350 5650 0    50   ~ 0
 LOCK_RELEASE
@@
 Wire Wire Line
 	8450 4500 9500 4500
+$Comp
+L Device:Q_NMOS_GDS Q1
+U 1 1 5D3AEAEC
+P 5250 6150
+F 0 "Q1" H 5456 6196 50  0000 L CNN
+F 1 "Q_NMOS_GDS" H 5456 6105 50  0000 L CNN
+F 2 "Package_TO_SOT_SMD:TO-252-3_TabPin2" H 5450 6250 50  0001 C CNN
+F 3 "~" H 5250 6150 50  0001 C CNN
+	1    5250 6150
+	1    0    0    -1
+$EndComp
 $EndSCHEMATC
